Commit message: huge platform

File: alunka_description/urdf/alunka_robot.urdf.xacro (robot description, xacro)
@@ -3,7 +3,7 @@
     <xacro:include filename="common_properties.xacro" />
     <xacro:include filename="mobile_robot.xacro" />
-    <xacro:include filename="balance_robot.xacro" />
-    <xacro:include filename="platform.xacro" />
-    <xacro:include filename="mobile_robot_gazebo.xacro" />
+    <!-- <xacro:include filename="balance_robot.xacro" /> -->
+    <!-- <xacro:include filename="platform.xacro" /> -->
+    <!-- <xacro:include filename="mobile_robot_gazebo.xacro" /> -->
     <!-- <xacro:include filename="camera.xacro" /> -->
 </robot>

File: alunka_description/urdf/balance_robot.xacro (robot description, xacro)
@@ -2,5 +2,5 @@
 <robot xmlns:xacro="http://www.ros.org/wiki/xacro">
     <xacro:property name="cylinder_radius" value="0.03" />
-    <xacro:property name="cylinder_lenght" value="0.5" />
+    <xacro:property name="cylinder_lenght" value="0.25" />
     <xacro:property name="small_cylinder_radius" value="0.02" />
     <xacro:property name="small_cylinder_lenght" value="${cylinder_lenght}" />

File: alunka_description/urdf/platform.xacro (robot description, xacro)
@@ -4,5 +4,5 @@
         <visual>
             <geometry>
-                <box size="${base_lenght} ${base_width} ${base_height / 4.0}" />
+                <box size="${base_lenght + 8} ${base_width+ 8} ${base_height / 4.0+ 8}" />
             </geometry>
             <origin xyz="${-base_lenght/2} 0 0" rpy="0 0 0" />
